Commit message: description/colors.xacro: Added brass color for spacers

File: description/colors.xacro (robot description, xacro)
@@ -6,4 +6,7 @@
   <material name="blue">
     <color rgba="0 0 1 1"/>
+  </material>
+  <material name="brass">
+    <color rgba="0.71, 0.651, 0.259 1"/>
   </material>
   <material name="green">
