Commit message: description/ros2_control.xacro: Rename var change conditional remove plugin
- Renamed variable to control which hardware interface to use
- Added conditionals for robot, mock, and gazebo to control respective
  hardware interfaces for each
- Removed gazebo plugin, in its own file included if that conditional is set
- Added additional parameters for wheel joints

File: description/ros2_control.xacro (robot description, xacro)
@@ -1,48 +1,61 @@
 <?xml version="1.0"?>
 <robot xmlns:xacro="http://www.ros.org/wiki/xacro">
-  <xacro:macro name="ros2_control" params="use_mock_hardware">
+  <xacro:macro name="ros2_control" params="use_hardware">
     <ros2_control name="ros2_control" type="system">
-       <xacro:unless value="${use_mock_hardware}">
+       <xacro:if value="${use_hardware == 'robot'}">
             <hardware>
-                <plugin>turbopi_hardware_interface/TurboPiSystemHardware</plugin>
+                <plugin>robot_hardware_interface/RobotSystemHardware</plugin>
                 <param name="hw_start_duration_sec">1.0</param>
                 <param name="hw_stop_duration_sec">3.0</param>
             </hardware>
-        </xacro:unless>
-        <xacro:if value="${use_mock_hardware}">
+        </xacro:if>
+        <xacro:if value="${use_hardware == 'mock'}">
+            <hardware>
+                <plugin>mock_components/GenericSystem</plugin>
+                <param name="calculate_dynamics">true</param>
+            </hardware>
+        </xacro:if>
+        <xacro:if value="${use_hardware == 'ign_gazebo'}">
             <hardware>
                 <plugin>gz_ros2_control/GazeboSimSystem</plugin>
-                <!-- <plugin>mock_components/GenericSystem</plugin>
-                <param name="calculate_dynamics">true</param> -->
             </hardware>
         </xacro:if>
         <joint name="front_left_wheel_joint">
             <command_interface name="velocity" />
-            <state_interface name="position" />
-            <state_interface name="velocity" />
+            <state_interface name="position">
+                <param name="initial_value">0</param>
+            </state_interface>
+            <state_interface name="velocity">
+                <param name="initial_value">0.0</param>
+            </state_interface>
         </joint>
         <joint name="front_right_wheel_joint">
             <command_interface name="velocity" />
-            <state_interface name="position" />
-            <state_interface name="velocity" />
+            <state_interface name="position">
+                <param name="initial_value">0</param>
+            </state_interface>
+            <state_interface name="velocity">
+                <param name="initial_value">0.0</param>
+            </state_interface>
         </joint>
         <joint name="rear_left_wheel_joint">
             <command_interface name="velocity" />
-            <state_interface name="position" />
-            <state_interface name="velocity" />
+            <state_interface name="position">
+                <param name="initial_value">0</param>
+            </state_interface>
+            <state_interface name="velocity">
+                <param name="initial_value">0.0</param>
+            </state_interface>
         </joint>
         <joint name="rear_right_wheel_joint">
             <command_interface name="velocity" />
-            <state_interface name="position" />
-            <state_interface name="velocity" />
+            <state_interface name="position">
+                <param name="initial_value">0</param>
+            </state_interface>
+            <state_interface name="velocity">
+                <param name="initial_value">0.0</param>
+            </state_interface>
         </joint>
     </ros2_control>
   </xacro:macro>
-    <gazebo>
-        <plugin filename="libgz_ros2_control-system.so" name="gz_ros2_control::GazeboSimROS2ControlPlugin">
-            <robot_param>robot_description</robot_param>
-            <robot_param_node>robot_state_publisher</robot_param_node>
-            <parameters>$(find turbopi_ros)/config/turbopi_controllers.yaml</parameters>
-        </plugin>
-    </gazebo>
 </robot>

Commit message: description/ros2_control.xacro: Added camera joints with limits & position

File: description/ros2_control.xacro (robot description, xacro)
@@ -57,4 +57,22 @@
             </state_interface>
         </joint>
+        <joint name="camera_joint">
+            <command_interface name="position">
+                <param name="min">-0.5</param>
+                <param name="max">1</param>
+            </command_interface>
+            <state_interface name="position">
+                <param name="initial_value">0</param>
+            </state_interface>
+        </joint>
+        <joint name="camera_frame_joint">
+            <command_interface name="position">
+                <param name="min">-1</param>
+                <param name="max">1</param>
+            </command_interface>
+            <state_interface name="position">
+                <param name="initial_value">0</param>
+            </state_interface>
+        </joint>
     </ros2_control>
   </xacro:macro>

Commit message: description/ros2_control.xacro: Wrap camera joints in style macro
- Initial work to control 2d camera and sonar or other
- Change nesting order of other macro

File: description/ros2_control.xacro (robot description, xacro)
@@ -1,24 +1,25 @@
 <?xml version="1.0"?>
 <robot xmlns:xacro="http://www.ros.org/wiki/xacro">
-  <xacro:macro name="ros2_control" params="use_hardware">
     <ros2_control name="ros2_control" type="system">
-       <xacro:if value="${use_hardware == 'robot'}">
-            <hardware>
-                <plugin>turbopi_hardware_interface/TurboPiSystemHardware</plugin>
-                <param name="hw_start_duration_sec">1.0</param>
-                <param name="hw_stop_duration_sec">3.0</param>
-            </hardware>
-        </xacro:if>
-        <xacro:if value="${use_hardware == 'mock'}">
-            <hardware>
-                <plugin>mock_components/GenericSystem</plugin>
-                <param name="calculate_dynamics">true</param>
-            </hardware>
-        </xacro:if>
-        <xacro:if value="${use_hardware == 'ign_gazebo'}">
-            <hardware>
-                <plugin>gz_ros2_control/GazeboSimSystem</plugin>
-            </hardware>
-        </xacro:if>
+        <xacro:macro name="ros2_control" params="use_hardware">
+            <xacro:if value="${use_hardware == 'robot'}">
+                <hardware>
+                    <plugin>turbopi_hardware_interface/TurboPiSystemHardware</plugin>
+                    <param name="hw_start_duration_sec">1.0</param>
+                    <param name="hw_stop_duration_sec">3.0</param>
+                </hardware>
+            </xacro:if>
+            <xacro:if value="${use_hardware == 'mock'}">
+                <hardware>
+                    <plugin>mock_components/GenericSystem</plugin>
+                    <param name="calculate_dynamics">true</param>
+                </hardware>
+            </xacro:if>
+            <xacro:if value="${use_hardware == 'ign_gazebo'}">
+                <hardware>
+                    <plugin>gz_ros2_control/GazeboSimSystem</plugin>
+                </hardware>
+            </xacro:if>
+        </xacro:macro>
         <joint name="front_left_wheel_joint">
             <command_interface name="velocity" />
@@ -57,23 +58,26 @@
             </state_interface>
         </joint>
-        <joint name="camera_joint">
-            <command_interface name="position">
-                <param name="min">-0.5</param>
-                <param name="max">1</param>
-            </command_interface>
-            <state_interface name="position">
-                <param name="initial_value">0</param>
-            </state_interface>
-        </joint>
-        <joint name="camera_frame_joint">
-            <command_interface name="position">
-                <param name="min">-1</param>
-                <param name="max">1</param>
-            </command_interface>
-            <state_interface name="position">
-                <param name="initial_value">0</param>
-            </state_interface>
-        </joint>
+        <xacro:macro name="style" params="use_style">
+            <xacro:if value="${use_style == 'default'}">
+                <joint name="camera_joint">
+                    <command_interface name="position">
+                        <param name="min">-0.5</param>
+                        <param name="max">1</param>
+                    </command_interface>
+                    <state_interface name="position">
+                        <param name="initial_value">0</param>
+                    </state_interface>
+                </joint>
+                <joint name="camera_frame_joint">
+                    <command_interface name="position">
+                        <param name="min">-1</param>
+                        <param name="max">1</param>
+                    </command_interface>
+                    <state_interface name="position">
+                        <param name="initial_value">0</param>
+                    </state_interface>
+                </joint>
+            </xacro:if>
+        </xacro:macro>
     </ros2_control>
-  </xacro:macro>
 </robot>

Commit message: description/ros2_control.xacro: Correct macro nesting and params usage

File: description/ros2_control.xacro (robot description, xacro)
@@ -1,6 +1,6 @@
 <?xml version="1.0"?>
 <robot xmlns:xacro="http://www.ros.org/wiki/xacro">
-    <ros2_control name="ros2_control" type="system">
-        <xacro:macro name="ros2_control" params="use_hardware">
+    <xacro:macro name="ros2_control" params="use_hardware use_style">
+        <ros2_control name="ros2_control" type="system">
             <xacro:if value="${use_hardware == 'robot'}">
                 <hardware>
@@ -21,42 +21,40 @@
                 </hardware>
             </xacro:if>
-        </xacro:macro>
-        <joint name="front_left_wheel_joint">
-            <command_interface name="velocity" />
-            <state_interface name="position">
-                <param name="initial_value">0</param>
-            </state_interface>
-            <state_interface name="velocity">
-                <param name="initial_value">0.0</param>
-            </state_interface>
-        </joint>
-        <joint name="front_right_wheel_joint">
-            <command_interface name="velocity" />
-            <state_interface name="position">
-                <param name="initial_value">0</param>
-            </state_interface>
-            <state_interface name="velocity">
-                <param name="initial_value">0.0</param>
-            </state_interface>
-        </joint>
-        <joint name="rear_left_wheel_joint">
-            <command_interface name="velocity" />
-            <state_interface name="position">
-                <param name="initial_value">0</param>
-            </state_interface>
-            <state_interface name="velocity">
-                <param name="initial_value">0.0</param>
-            </state_interface>
-        </joint>
-        <joint name="rear_right_wheel_joint">
-            <command_interface name="velocity" />
-            <state_interface name="position">
-                <param name="initial_value">0</param>
-            </state_interface>
-            <state_interface name="velocity">
-                <param name="initial_value">0.0</param>
-            </state_interface>
-        </joint>
-        <xacro:macro name="style" params="use_style">
+            <joint name="front_left_wheel_joint">
+                <command_interface name="velocity" />
+                <state_interface name="position">
+                    <param name="initial_value">0</param>
+                </state_interface>
+                <state_interface name="velocity">
+                    <param name="initial_value">0.0</param>
+                </state_interface>
+            </joint>
+            <joint name="front_right_wheel_joint">
+                <command_interface name="velocity" />
+                <state_interface name="position">
+                    <param name="initial_value">0</param>
+                </state_interface>
+                <state_interface name="velocity">
+                    <param name="initial_value">0.0</param>
+                </state_interface>
+            </joint>
+            <joint name="rear_left_wheel_joint">
+                <command_interface name="velocity" />
+                <state_interface name="position">
+                    <param name="initial_value">0</param>
+                </state_interface>
+                <state_interface name="velocity">
+                    <param name="initial_value">0.0</param>
+                </state_interface>
+            </joint>
+            <joint name="rear_right_wheel_joint">
+                <command_interface name="velocity" />
+                <state_interface name="position">
+                    <param name="initial_value">0</param>
+                </state_interface>
+                <state_interface name="velocity">
+                    <param name="initial_value">0.0</param>
+                </state_interface>
+            </joint>
             <xacro:if value="${use_style == 'default'}">
                 <joint name="camera_joint">
@@ -79,5 +77,5 @@
                 </joint>
             </xacro:if>
-        </xacro:macro>
-    </ros2_control>
+        </ros2_control>
+    </xacro:macro>
 </robot>

Commit message: description/ros2_control.xacro: Rename style/use_style to camera/use_camera

File: description/ros2_control.xacro (robot description, xacro)
@@ -1,5 +1,5 @@
 <?xml version="1.0"?>
 <robot xmlns:xacro="http://www.ros.org/wiki/xacro">
-    <xacro:macro name="ros2_control" params="use_hardware use_style">
+    <xacro:macro name="ros2_control" params="use_hardware use_camera">
         <ros2_control name="ros2_control" type="system">
             <xacro:if value="${use_hardware == 'robot'}">
@@ -57,5 +57,5 @@
                 </state_interface>
             </joint>
-            <xacro:if value="${use_style == 'default'}">
+            <xacro:if value="${use_camera == 'default'}">
                 <joint name="camera_joint">
                     <command_interface name="position">
