Commit message: description/turbopi_core.xacro: Added collision tags

File: description/turbopi_core.xacro (robot description, xacro)
@@ -8,4 +8,10 @@
     </joint>
     <link name="chassis">
+        <collision>
+            <origin xyz="0.0935 0 0.00" rpy="0 0 0"/>
+            <geometry>
+                <box size="0.187 0.095 0.04"/>
+            </geometry>
+        </collision>
         <visual>
             <origin xyz="0.0935 0 0.00" rpy="0 0 0"/>
@@ -24,4 +30,9 @@
     </joint>
     <link name="front_left_wheel">
+        <collision>
+            <geometry>
+                <cylinder length="0.03" radius="0.0325" />
+            </geometry>
+        </collision>
         <visual>
             <geometry>
@@ -39,4 +50,9 @@
     </joint>
     <link name="front_right_wheel">
+        <collision>
+            <geometry>
+                <cylinder length="0.03" radius="0.0325" />
+            </geometry>
+        </collision>
         <visual>
             <geometry>
@@ -54,4 +70,9 @@
     </joint>
     <link name="rear_left_wheel">
+        <collision>
+            <geometry>
+                <cylinder length="0.03" radius="0.0325" />
+            </geometry>
+        </collision>
         <visual>
             <geometry>
@@ -69,4 +90,9 @@
     </joint>
     <link name="rear_right_wheel">
+        <collision>
+            <geometry>
+                <cylinder length="0.03" radius="0.0325" />
+            </geometry>
+        </collision>
         <visual>
             <geometry>

Commit message: description/turbopi_core.xacro: Include inertial macros

File: description/turbopi_core.xacro (robot description, xacro)
@@ -21,4 +21,7 @@
             <material name="white"/>
         </visual>
+        <xacro:inertial_box mass="0.5" x="0.187" y="0.095" z="0.04">
+            <origin xyz="0.0935 0 0.04675" rpy="0 0 0"/>
+        </xacro:inertial_box>
     </link>
     <!-- Front Left Wheel -->
@@ -41,4 +44,7 @@
             <material name="yellow"/>
         </visual>
+        <xacro:inertial_cylinder mass="0.1" length="0.03" radius="0.0325">
+            <origin xyz="0 0 0" rpy="0 0 0"/>
+        </xacro:inertial_cylinder>
     </link>
     <!-- Front Right Wheel -->
@@ -61,4 +67,7 @@
             <material name="yellow"/>
         </visual>
+        <xacro:inertial_cylinder mass="0.1" length="0.03" radius="0.0325">
+            <origin xyz="0 0 0" rpy="0 0 0"/>
+        </xacro:inertial_cylinder>
     </link>
     <!-- Rear Left Wheel -->
@@ -81,4 +90,7 @@
             <material name="yellow"/>
         </visual>
+        <xacro:inertial_cylinder mass="0.1" length="0.03" radius="0.0325">
+            <origin xyz="0 0 0" rpy="0 0 0"/>
+        </xacro:inertial_cylinder>
     </link>
     <!-- Rear Right Wheel -->
@@ -101,4 +113,7 @@
             <material name="yellow"/>
         </visual>
+        <xacro:inertial_cylinder mass="0.1" length="0.03" radius="0.0325">
+            <origin xyz="0 0 0" rpy="0 0 0"/>
+        </xacro:inertial_cylinder>
     </link>
 </robot>

Commit message: description/turbopi_core.xacro: Added limit tags

File: description/turbopi_core.xacro (robot description, xacro)
@@ -31,4 +31,5 @@
         <origin xyz="-0.0585 0.0725 0" rpy="-${pi/2} 0 0"/>
         <axis xyz="0 0 1"/>
+        <limit effort="100.0" lower="-100" upper="100" velocity="1"/>
     </joint>
     <link name="front_left_wheel">
@@ -54,4 +55,5 @@
         <origin xyz="-0.0585 -0.0725 0" rpy="${pi/2} 0 0"/>
         <axis xyz="0 0 -1"/>
+        <limit effort="100.0" lower="-100" upper="100" velocity="1"/>
     </joint>
     <link name="front_right_wheel">
@@ -77,4 +79,5 @@
         <origin xyz="0.062 0.0725 0" rpy="-${pi/2} 0 0"/>
         <axis xyz="0 0 1"/>
+        <limit effort="100.0" lower="-100" upper="100" velocity="1"/>
     </joint>
     <link name="rear_left_wheel">
@@ -100,4 +103,5 @@
         <origin xyz="0.062 -0.0725 0" rpy="${pi/2} 0 0"/>
         <axis xyz="0 0 -1"/>
+        <limit effort="100.0" lower="-100" upper="100" velocity="1"/>
     </joint>
     <link name="rear_right_wheel">

Commit message: description/turbopi_core.xacro: Replaced values with variables initial work
- The wheels are not properly aligned, as they will be replaced with mesh

File: description/turbopi_core.xacro (robot description, xacro)
@@ -1,49 +1,62 @@
 <?xml version="1.0"?>
 <robot xmlns:xacro="http://www.ros.org/wiki/xacro">
+    <xacro:property name="collision_multiplier" value="1.5" />
+    <xacro:property name="limit_effort" value="100" />
+    <xacro:property name="limit_velocity" value="10" />
+    <xacro:property name="chassis_length" value="0.187" />
+    <xacro:property name="chassis_height" value="0.04" />
+    <xacro:property name="chassis_width" value="0.095" />
+    <xacro:property name="wheel_gap" value="0.001" />
+    <xacro:property name="wheel_length" value="0.03" />
+    <xacro:property name="wheel_radius" value="0.0325" />
+    <xacro:property name="wheel_mass" value="0.0016" />
+    <xacro:property name="wheel_offset_front" value="${-chassis_length/2 + 0.1778}" />
+    <xacro:property name="wheel_offset_rear" value="${chassis_length/2 - 0.2286}" />
+    <xacro:property name="wheel_offset_side" value="${wheel_length/2 + chassis_width/2 + wheel_gap}" />
     <link name="base_link"></link>
+    <!-- Main Body/Chassis -->
     <joint name="chassis_joint" type="fixed">
         <parent link="base_link"/>
         <child link="chassis"/>
-        <origin xyz="-0.1 0 0"/>
+        <origin xyz="0 0 ${wheel_radius}" rpy="0 0 0"/>
     </joint>
     <link name="chassis">
         <collision>
-            <origin xyz="0.0935 0 0.00" rpy="0 0 0"/>
             <geometry>
-                <box size="0.187 0.095 0.04"/>
+                <box size="${chassis_length * collision_multiplier} ${chassis_width} ${chassis_height}"/>
             </geometry>
         </collision>
         <visual>
-            <origin xyz="0.0935 0 0.00" rpy="0 0 0"/>
             <geometry>
-                <box size="0.187 0.095 0.04"/>
+                <box size="${chassis_length} ${chassis_width} ${chassis_height}"/>
             </geometry>
             <material name="white"/>
         </visual>
-        <xacro:inertial_box mass="0.5" x="0.187" y="0.095" z="0.04">
-            <origin xyz="0.0935 0 0.04675" rpy="0 0 0"/>
+        <xacro:inertial_box mass="0.5" x="${chassis_length}" y="${chassis_width}" z="${chassis_height}">
+            <origin xyz="0 0 0" rpy="0 0 0"/>
         </xacro:inertial_box>
     </link>
     <!-- Front Left Wheel -->
     <joint name="front_left_wheel_joint" type="continuous">
-        <parent link="base_link"/>
+        <parent link="chassis"/>
         <child link="front_left_wheel"/>
-        <origin xyz="-0.0585 0.0725 0" rpy="-${pi/2} 0 0"/>
+        <origin xyz="${wheel_offset_front} ${wheel_offset_side} 0" rpy="-${pi/2} 0 0"/>
         <axis xyz="0 0 1"/>
-        <limit effort="100.0" lower="-100" upper="100" velocity="1"/>
+        <limit effort="${limit_effort}" velocity="${limit_velocity}"/>
     </joint>
     <link name="front_left_wheel">
         <collision>
             <geometry>
-                <cylinder length="0.03" radius="0.0325" />
+                <cylinder length="${wheel_length * collision_multiplier}" radius="${wheel_radius}" />
             </geometry>
         </collision>
         <visual>
+            <origin xyz="-${wheel_radius} -${wheel_radius} ${wheel_length/2}" rpy="-${pi/2} 0 0"/>
             <geometry>
-                <cylinder length="0.03" radius="0.0325" />
+                <cylinder length="${wheel_length}" radius="${wheel_radius}" />
             </geometry>
             <material name="yellow"/>
         </visual>
-        <xacro:inertial_cylinder mass="0.1" length="0.03" radius="0.0325">
+        <xacro:inertial_cylinder mass="${wheel_mass}" length="${wheel_length}" radius="${wheel_radius}">
             <origin xyz="0 0 0" rpy="0 0 0"/>
         </xacro:inertial_cylinder>
@@ -51,23 +64,24 @@
     <!-- Front Right Wheel -->
     <joint name="front_right_wheel_joint" type="continuous">
-        <parent link="base_link"/>
+        <parent link="chassis"/>
         <child link="front_right_wheel"/>
-        <origin xyz="-0.0585 -0.0725 0" rpy="${pi/2} 0 0"/>
+        <origin xyz="${wheel_offset_front} -${wheel_offset_side} 0" rpy="${pi/2} 0 0"/>
         <axis xyz="0 0 -1"/>
-        <limit effort="100.0" lower="-100" upper="100" velocity="1"/>
+        <limit effort="${limit_effort}" velocity="${limit_velocity}"/>
     </joint>
     <link name="front_right_wheel">
         <collision>
             <geometry>
-                <cylinder length="0.03" radius="0.0325" />
+                <cylinder length="${wheel_length * collision_multiplier}" radius="${wheel_radius}" />
             </geometry>
         </collision>
         <visual>
+            <origin xyz="-${wheel_radius} ${wheel_radius} -${wheel_length/2}" rpy="${pi/2} 0 0"/>
             <geometry>
-                <cylinder length="0.03" radius="0.0325" />
+                <cylinder length="${wheel_length}" radius="${wheel_radius}" />
             </geometry>
             <material name="yellow"/>
         </visual>
-        <xacro:inertial_cylinder mass="0.1" length="0.03" radius="0.0325">
+        <xacro:inertial_cylinder mass="${wheel_mass}" length="${wheel_length}" radius="${wheel_radius}">
             <origin xyz="0 0 0" rpy="0 0 0"/>
         </xacro:inertial_cylinder>
@@ -75,23 +89,24 @@
     <!-- Rear Left Wheel -->
     <joint name="rear_left_wheel_joint" type="continuous">
-        <parent link="base_link"/>
+        <parent link="chassis"/>
         <child link="rear_left_wheel"/>
-        <origin xyz="0.062 0.0725 0" rpy="-${pi/2} 0 0"/>
+        <origin xyz="${wheel_offset_rear} ${wheel_offset_side} 0" rpy="-${pi/2} 0 0"/>
         <axis xyz="0 0 1"/>
-        <limit effort="100.0" lower="-100" upper="100" velocity="1"/>
+        <limit effort="${limit_effort}" velocity="${limit_velocity}"/>
     </joint>
     <link name="rear_left_wheel">
         <collision>
             <geometry>
-                <cylinder length="0.03" radius="0.0325" />
+                <cylinder length="${wheel_length * collision_multiplier}" radius="${wheel_radius}" />
             </geometry>
         </collision>
         <visual>
+            <origin xyz="-${wheel_radius} -${wheel_radius} ${wheel_length/2}" rpy="-${pi/2} 0 0"/>
             <geometry>
-                <cylinder length="0.03" radius="0.0325" />
+                <cylinder length="${wheel_length}" radius="${wheel_radius}" />
             </geometry>
             <material name="yellow"/>
         </visual>
-        <xacro:inertial_cylinder mass="0.1" length="0.03" radius="0.0325">
+        <xacro:inertial_cylinder mass="${wheel_mass}" length="${wheel_length}" radius="${wheel_radius}">
             <origin xyz="0 0 0" rpy="0 0 0"/>
         </xacro:inertial_cylinder>
@@ -99,23 +114,24 @@
     <!-- Rear Right Wheel -->
     <joint name="rear_right_wheel_joint" type="continuous">
-        <parent link="base_link"/>
+        <parent link="chassis"/>
         <child link="rear_right_wheel"/>
-        <origin xyz="0.062 -0.0725 0" rpy="${pi/2} 0 0"/>
+        <origin xyz="${wheel_offset_rear} -${wheel_offset_side} 0" rpy="${pi/2} 0 0"/>
         <axis xyz="0 0 -1"/>
-        <limit effort="100.0" lower="-100" upper="100" velocity="1"/>
+        <limit effort="${limit_effort}" velocity="${limit_velocity}"/>
     </joint>
     <link name="rear_right_wheel">
         <collision>
             <geometry>
-                <cylinder length="0.03" radius="0.0325" />
+                <cylinder length="${wheel_length * collision_multiplier}" radius="${wheel_radius}" />
             </geometry>
         </collision>
         <visual>
+            <origin xyz="-${wheel_radius} ${wheel_radius} -${wheel_length/2}" rpy="${pi/2} 0 0"/>
             <geometry>
-                <cylinder length="0.03" radius="0.0325" />
+                <cylinder length="${wheel_length}" radius="${wheel_radius}" />
             </geometry>
             <material name="yellow"/>
         </visual>
-        <xacro:inertial_cylinder mass="0.1" length="0.03" radius="0.0325">
+        <xacro:inertial_cylinder mass="${wheel_mass}" length="${wheel_length}" radius="${wheel_radius}">
             <origin xyz="0 0 0" rpy="0 0 0"/>
         </xacro:inertial_cylinder>

Commit message: description/turbopi_core.xacro: Initial mesh files for chassis & wheels
- Modified variable values, added new ones, and added mesh files

File: description/turbopi_core.xacro (robot description, xacro)
@@ -6,12 +6,15 @@
     <xacro:property name="chassis_length" value="0.187" />
     <xacro:property name="chassis_height" value="0.04" />
-    <xacro:property name="chassis_width" value="0.095" />
-    <xacro:property name="wheel_gap" value="0.001" />
+    <xacro:property name="chassis_width" value="0.094" />
+    <xacro:property name="mesh_scale" value="0.001 0.001 0.001" />
+    <xacro:property name="wheel_gap" value="0.005" />
     <xacro:property name="wheel_length" value="0.03" />
     <xacro:property name="wheel_radius" value="0.0325" />
     <xacro:property name="wheel_mass" value="0.0016" />
-    <xacro:property name="wheel_offset_front" value="${-chassis_length/2 + 0.1778}" />
-    <xacro:property name="wheel_offset_rear" value="${chassis_length/2 - 0.2286}" />
+    <xacro:property name="wheel_mesh_file" value="file://$(find turbopi_ros)/meshes/wheel.dae" />
+    <xacro:property name="wheel_offset_front" value="${-chassis_length/2 + 0.0372}" />
+    <xacro:property name="wheel_offset_rear" value="${chassis_length/2 - 0.0305}" />
     <xacro:property name="wheel_offset_side" value="${wheel_length/2 + chassis_width/2 + wheel_gap}" />
+    <xacro:property name="wheel_zoffset" value="${chassis_height/2 + 0.0064}" />
     <link name="base_link"></link>
     <!-- Main Body/Chassis -->
@@ -19,5 +22,5 @@
         <parent link="base_link"/>
         <child link="chassis"/>
-        <origin xyz="0 0 ${wheel_radius}" rpy="0 0 0"/>
+        <origin xyz="0 0 ${wheel_radius + chassis_height/2}" rpy="0 0 0"/>
     </joint>
     <link name="chassis">
@@ -29,5 +32,5 @@
         <visual>
             <geometry>
-                <box size="${chassis_length} ${chassis_width} ${chassis_height}"/>
+                <mesh filename="file://$(find turbopi_ros)/meshes/chassis.dae" scale="${mesh_scale}" />
             </geometry>
             <material name="white"/>
@@ -41,5 +44,5 @@
         <parent link="chassis"/>
         <child link="front_left_wheel"/>
-        <origin xyz="${wheel_offset_front} ${wheel_offset_side} 0" rpy="-${pi/2} 0 0"/>
+        <origin xyz="${wheel_offset_front} -${wheel_offset_side} -${wheel_zoffset}" rpy="${pi/2} ${pi/2} 0"/>
         <axis xyz="0 0 1"/>
         <limit effort="${limit_effort}" velocity="${limit_velocity}"/>
@@ -52,7 +55,7 @@
         </collision>
         <visual>
-            <origin xyz="-${wheel_radius} -${wheel_radius} ${wheel_length/2}" rpy="-${pi/2} 0 0"/>
+            <origin xyz="0 0 0" rpy="-${pi/2} 0 0"/>
             <geometry>
-                <cylinder length="${wheel_length}" radius="${wheel_radius}" />
+                <mesh filename="${wheel_mesh_file}" scale="${mesh_scale}" />
             </geometry>
             <material name="yellow"/>
@@ -66,5 +69,5 @@
         <parent link="chassis"/>
         <child link="front_right_wheel"/>
-        <origin xyz="${wheel_offset_front} -${wheel_offset_side} 0" rpy="${pi/2} 0 0"/>
+        <origin xyz="${wheel_offset_front} ${wheel_offset_side} -${wheel_zoffset}" rpy="-${pi/2} ${pi/2} 0"/>
         <axis xyz="0 0 -1"/>
         <limit effort="${limit_effort}" velocity="${limit_velocity}"/>
@@ -77,7 +80,7 @@
         </collision>
         <visual>
-            <origin xyz="-${wheel_radius} ${wheel_radius} -${wheel_length/2}" rpy="${pi/2} 0 0"/>
+            <origin xyz="0 0 0" rpy="-${pi/2} 0 0"/>
             <geometry>
-                <cylinder length="${wheel_length}" radius="${wheel_radius}" />
+                <mesh filename="${wheel_mesh_file}" scale="${mesh_scale}" />
             </geometry>
             <material name="yellow"/>
@@ -91,5 +94,5 @@
         <parent link="chassis"/>
         <child link="rear_left_wheel"/>
-        <origin xyz="${wheel_offset_rear} ${wheel_offset_side} 0" rpy="-${pi/2} 0 0"/>
+        <origin xyz="${wheel_offset_rear} -${wheel_offset_side} -${wheel_zoffset}" rpy="${pi/2} ${pi/2} 0"/>
         <axis xyz="0 0 1"/>
         <limit effort="${limit_effort}" velocity="${limit_velocity}"/>
@@ -102,7 +105,7 @@
         </collision>
         <visual>
-            <origin xyz="-${wheel_radius} -${wheel_radius} ${wheel_length/2}" rpy="-${pi/2} 0 0"/>
+            <origin xyz="0 0 0" rpy="-${pi/2} 0 0"/>
             <geometry>
-                <cylinder length="${wheel_length}" radius="${wheel_radius}" />
+                <mesh filename="${wheel_mesh_file}" scale="${mesh_scale}" />
             </geometry>
             <material name="yellow"/>
@@ -116,5 +119,5 @@
         <parent link="chassis"/>
         <child link="rear_right_wheel"/>
-        <origin xyz="${wheel_offset_rear} -${wheel_offset_side} 0" rpy="${pi/2} 0 0"/>
+        <origin xyz="${wheel_offset_rear} ${wheel_offset_side} -${wheel_zoffset}" rpy="-${pi/2} ${pi/2} 0"/>
         <axis xyz="0 0 -1"/>
         <limit effort="${limit_effort}" velocity="${limit_velocity}"/>
@@ -127,7 +130,7 @@
         </collision>
         <visual>
-            <origin xyz="-${wheel_radius} ${wheel_radius} -${wheel_length/2}" rpy="${pi/2} 0 0"/>
+            <origin xyz="0 0 0" rpy="-${pi/2} 0 0"/>
             <geometry>
-                <cylinder length="${wheel_length}" radius="${wheel_radius}" />
+                <mesh filename="${wheel_mesh_file}" scale="${mesh_scale}" />
             </geometry>
             <material name="yellow"/>

Commit message: description/turbopi_core.xacro: Added camera frame, initial origin & size

File: description/turbopi_core.xacro (robot description, xacro)
@@ -4,4 +4,7 @@
     <xacro:property name="limit_effort" value="100" />
     <xacro:property name="limit_velocity" value="10" />
+    <xacro:property name="camera_frame_length" value="0.0254" />
+    <xacro:property name="camera_frame_height" value="0.0333" />
+    <xacro:property name="camera_frame_width" value="0.04445" />
     <xacro:property name="chassis_length" value="0.187" />
     <xacro:property name="chassis_height" value="0.04" />
@@ -140,3 +143,27 @@
         </xacro:inertial_cylinder>
     </link>
+    <!-- Camera frame turns left/right -->
+    <joint name="camera_frame_joint" type="revolute">
+        <parent link="chassis"/>
+        <child link="camera_frame"/>
+        <origin xyz="${-chassis_length/2 + 0.054} 0 ${chassis_height + 0.01}" rpy="0 0 0"/>
+        <limit lower="-90"  upper="90"  velocity="0.1"  effort="${limit_effort}"  />
+        <axis xyz="0 0 1"/>
+    </joint>
+    <link name="camera_frame">
+        <collision>
+            <geometry>
+                <box size="${camera_frame_length} ${camera_frame_width} ${camera_frame_height}"/>
+            </geometry>
+        </collision>
+        <visual>
+            <geometry>
+                <mesh filename="file://$(find turbopi_ros)/meshes/camera_frame.dae" scale="${mesh_scale}" />
+            </geometry>
+            <material name="white"/>
+        </visual>
+        <xacro:inertial_box mass="0.01" x="${camera_frame_length}" y="${camera_frame_width}" z="${camera_frame_height}">
+            <origin xyz="0 0 ${camera_frame_height/2}" rpy="0 0 0"/>
+        </xacro:inertial_box>
+    </link>
 </robot>

Commit message: description/turbopi_core.xacro: Added camera, initial origin & size

File: description/turbopi_core.xacro (robot description, xacro)
@@ -4,4 +4,7 @@
     <xacro:property name="limit_effort" value="100" />
     <xacro:property name="limit_velocity" value="10" />
+    <xacro:property name="camera_length" value="0.0635" />
+    <xacro:property name="camera_height" value="0.03175" />
+    <xacro:property name="camera_width" value="0.0333" />
     <xacro:property name="camera_frame_length" value="0.0254" />
     <xacro:property name="camera_frame_height" value="0.0333" />
@@ -167,3 +170,27 @@
         </xacro:inertial_box>
     </link>
+    <!-- Camera angles up/down -->
+    <joint name="camera_joint" type="revolute">
+        <parent link="camera_frame"/>
+        <child link="camera"/>
+        <origin xyz="-0.015 0 ${camera_frame_height * 0.4}" rpy="0 0 0"/>
+        <limit lower="-45"  upper="90"  velocity="0.1"  effort="${limit_effort}"  />
+        <axis xyz="0 0 1"/>
+    </joint>
+    <link name="camera">
+        <collision>
+            <geometry>
+                <box size="${camera_length} ${camera_width} ${camera_height}"/>
+            </geometry>
+        </collision>
+        <visual>
+            <geometry>
+                <mesh filename="file://$(find turbopi_ros)/meshes/camera.dae" scale="${mesh_scale}" />
+            </geometry>
+            <material name="white"/>
+        </visual>
+        <xacro:inertial_box mass="0.01" x="${camera_length}" y="${camera_width}" z="${camera_height}">
+            <origin xyz="0 0 ${camera_height/2}" rpy="0 0 0"/>
+        </xacro:inertial_box>
+    </link>
 </robot>

Commit message: description/turbopi_core.xacro: Modify/correct limits for camera joints

File: description/turbopi_core.xacro (robot description, xacro)
@@ -151,5 +151,5 @@
         <child link="camera_frame"/>
         <origin xyz="${-chassis_length/2 + 0.054} 0 ${chassis_height + 0.01}" rpy="0 0 0"/>
-        <limit lower="-90"  upper="90"  velocity="0.1"  effort="${limit_effort}"  />
+        <limit lower="-1"  upper="1"  velocity="0.1"  effort="${limit_effort}"  />
         <axis xyz="0 0 1"/>
     </joint>
@@ -175,6 +175,6 @@
         <child link="camera"/>
         <origin xyz="-0.015 0 ${camera_frame_height * 0.4}" rpy="0 0 0"/>
-        <limit lower="-45"  upper="90"  velocity="0.1"  effort="${limit_effort}"  />
-        <axis xyz="0 0 1"/>
+        <limit lower="-0.5"  upper="1"  velocity="0.1"  effort="${limit_effort}"  />
+        <axis xyz="0 1 0"/>
     </joint>
     <link name="camera">
