Commit message: description/turbopi_core.xacro: Added standoff spacers for the rear deck
- Visual only, so the rear deck is not floating...

File: description/turbopi_core.xacro (robot description, xacro)
@@ -14,4 +14,8 @@
     <xacro:property name="chassis_width" value="0.094" />
     <xacro:property name="mesh_scale" value="0.001 0.001 0.001" />
+    <xacro:property name="spacer_offset_front" value="0.0203" />
+    <xacro:property name="spacer_offset_rear" value="${chassis_width - 0.0135}" />
+    <xacro:property name="spacer_offset_side" value="${chassis_width/2 - 0.0138}" />
+    <xacro:property name="spacer_offset_height" value="0.015" />
     <xacro:property name="wheel_gap" value="0.005" />
     <xacro:property name="wheel_length" value="0.03" />
@@ -46,4 +50,56 @@
         </xacro:inertial_box>
     </link>
+    <joint name="spacer_1_joint" type="fixed">
+        <parent link="chassis"/>
+        <child link="spacer_1"/>
+        <origin xyz="${spacer_offset_front} ${spacer_offset_side} ${spacer_offset_height}" rpy="0 0 0"/>
+    </joint>
+    <link name="spacer_1">
+        <visual>
+            <geometry>
+                <mesh filename="file://$(find turbopi_ros)/meshes/spacer.dae" scale="${mesh_scale}" />
+            </geometry>
+            <material name="brass"/>
+        </visual>
+    </link>
+    <joint name="spacer_2_joint" type="fixed">
+        <parent link="chassis"/>
+        <child link="spacer_2"/>
+        <origin xyz="${spacer_offset_front} -${spacer_offset_side} ${spacer_offset_height}" rpy="0 0 0"/>
+    </joint>
+    <link name="spacer_2">
+        <visual>
+            <geometry>
+                <mesh filename="file://$(find turbopi_ros)/meshes/spacer.dae" scale="${mesh_scale}" />
+            </geometry>
+            <material name="brass"/>
+        </visual>
+    </link>
+    <joint name="spacer_3_joint" type="fixed">
+        <parent link="chassis"/>
+        <child link="spacer_3"/>
+        <origin xyz="${spacer_offset_rear} ${spacer_offset_side} ${spacer_offset_height}" rpy="0 0 0"/>
+    </joint>
+    <link name="spacer_3">
+        <visual>
+            <geometry>
+                <mesh filename="file://$(find turbopi_ros)/meshes/spacer.dae" scale="${mesh_scale}" />
+            </geometry>
+            <material name="brass"/>
+        </visual>
+    </link>
+    <joint name="spacer_4_joint" type="fixed">
+        <parent link="chassis"/>
+        <child link="spacer_4"/>
+        <origin xyz="${spacer_offset_rear} -${spacer_offset_side} ${spacer_offset_height}" rpy="0 0 0"/>
+    </joint>
+    <link name="spacer_4">
+        <visual>
+            <geometry>
+                <mesh filename="file://$(find turbopi_ros)/meshes/spacer.dae" scale="${mesh_scale}" />
+            </geometry>
+            <material name="brass"/>
+        </visual>
+    </link>
     <!-- Front Left Wheel -->
     <joint name="front_left_wheel_joint" type="continuous">

Commit message: description/turbopi_core.xacro: Raise chassis slightly to prive rise in sim
- Robot is in the floor a bit in gazebo, need to raise the chassis height
  some to get it to not rise on simulation start

File: description/turbopi_core.xacro (robot description, xacro)
@@ -32,5 +32,5 @@
         <parent link="base_link"/>
         <child link="chassis"/>
-        <origin xyz="0 0 ${wheel_radius + chassis_height/2}" rpy="0 0 0"/>
+        <origin xyz="0 0 ${wheel_radius + chassis_height/2 + 0.0065}" rpy="0 0 0"/>
     </joint>
     <link name="chassis">

Commit message: description/turbopi_core.xacro: Roll pitch camera face forward vs backward
- Simulated camera is facing backwards, chassis and wheels might be reversed
  easier to roll pitch camera than to flip the robot model

File: description/turbopi_core.xacro (robot description, xacro)
@@ -230,5 +230,5 @@
         <parent link="camera_frame"/>
         <child link="camera"/>
-        <origin xyz="-0.015 0 ${camera_frame_height * 0.4}" rpy="0 0 0"/>
+        <origin xyz="-0.015 0 ${camera_frame_height * 0.4}" rpy="${pi} ${pi} 0"/>
         <limit lower="-0.5"  upper="1"  velocity="0.1"  effort="${limit_effort}"  />
         <axis xyz="0 1 0"/>
@@ -241,4 +241,5 @@
         </collision>
         <visual>
+            <origin xyz="0 0 0" rpy="${pi} ${pi} 0"/>
             <geometry>
                 <mesh filename="file://$(find turbopi_ros)/meshes/camera.dae" scale="${mesh_scale}" />

Commit message: description/turbopi_core.xacro: Added rplidar with mesh

File: description/turbopi_core.xacro (robot description, xacro)
@@ -13,4 +13,7 @@
     <xacro:property name="chassis_height" value="0.04" />
     <xacro:property name="chassis_width" value="0.094" />
+    <xacro:property name="lidar_length" value="0.12954" />
+    <xacro:property name="lidar_height" value="0.07874" />
+    <xacro:property name="lidar_width" value="0.09906" />
     <xacro:property name="mesh_scale" value="0.001 0.001 0.001" />
     <xacro:property name="spacer_offset_front" value="0.0203" />
@@ -251,3 +254,26 @@
         </xacro:inertial_box>
     </link>
+    <!-- 360 Lidar -->
+    <joint name="lidar_joint" type="fixed">
+        <parent link="chassis"/>
+        <child link="lidar"/>
+        <axis xyz="0 0 1"/>
+        <origin xyz="${lidar_length/2 - 0.01} 0 0.0725" rpy="0 0 0"/>
+    </joint>
+    <link name="lidar">
+        <collision>
+            <geometry>
+                <box size="${lidar_length} ${lidar_width} ${lidar_height}"/>
+            </geometry>
+        </collision>
+        <visual>
+            <geometry>
+                <mesh filename="file://$(find turbopi_ros)/meshes/rplidar.dae" scale="1 1 1" />
+            </geometry>
+            <material name="black"/>
+        </visual>
+        <xacro:inertial_box mass="0.01" x="${lidar_length}" y="${lidar_width}" z="${chassis_height}">
+            <origin xyz="0 0 0" rpy="0 0 0"/>
+        </xacro:inertial_box>
+    </link>
 </robot>

Commit message: description/turbopi_core.xacro: Added base_footprint_joint & base_footprint
- Used for odom & lidar to be on the ground vs the ground mid center of the
  chassis for maps, etc

File: description/turbopi_core.xacro (robot description, xacro)
@@ -31,4 +31,11 @@
     <xacro:property name="wheel_zoffset" value="${chassis_height/2 + 0.0064}" />
     <link name="base_link"></link>
+    <joint name="base_footprint_joint" type="fixed">
+        <parent link="base_link"/>
+        <child link="base_footprint"/>
+    </joint>
+    <link name="base_footprint">
+        <parent link="base_link"/>
+    </link>
     <!-- Main Body/Chassis -->
     <joint name="chassis_joint" type="fixed">

Commit message: description/turbopi_core.xacro: Added ultrasonic sonar sensor with mesh

File: description/turbopi_core.xacro (robot description, xacro)
@@ -17,4 +17,7 @@
     <xacro:property name="lidar_width" value="0.09906" />
     <xacro:property name="mesh_scale" value="0.001 0.001 0.001" />
+    <xacro:property name="sonar_length" value="0.0254" />
+    <xacro:property name="sonar_height" value="0.0254" />
+    <xacro:property name="sonar_width" value="0.0508" />
     <xacro:property name="spacer_offset_front" value="0.0203" />
     <xacro:property name="spacer_offset_rear" value="${chassis_width - 0.0135}" />
@@ -261,4 +264,27 @@
         </xacro:inertial_box>
     </link>
+    <!-- Sonar -->
+    <joint name="sonar_joint" type="fixed">
+        <parent link="chassis"/>
+        <child link="sonar"/>
+        <axis xyz="0 0 1"/>
+        <origin xyz="-${chassis_length/2 - sonar_length*0.8} 0 ${sonar_height/5}" rpy="0 0 0"/>
+    </joint>
+    <link name="sonar">
+        <collision>
+            <geometry>
+                <box size="${sonar_length} ${sonar_width} ${sonar_height}"/>
+            </geometry>
+        </collision>
+        <visual>
+            <geometry>
+                <mesh filename="file://$(find turbopi_ros)/meshes/sonar.dae" scale="${mesh_scale}" />
+            </geometry>
+            <material name="white"/>
+        </visual>
+        <xacro:inertial_box mass="0.01" x="${sonar_length}" y="${sonar_width}" z="${sonar_height}">
+            <origin xyz="0 0 0" rpy="0 0 0"/>
+        </xacro:inertial_box>
+    </link>
     <!-- 360 Lidar -->
     <joint name="lidar_joint" type="fixed">

Commit message: description/turbopi_core.xacro: Roll pitch sonar, robot might be backward?

File: description/turbopi_core.xacro (robot description, xacro)
@@ -269,5 +269,5 @@
         <child link="sonar"/>
         <axis xyz="0 0 1"/>
-        <origin xyz="-${chassis_length/2 - sonar_length*0.8} 0 ${sonar_height/5}" rpy="0 0 0"/>
+        <origin xyz="-${chassis_length/2 - sonar_length*0.8} 0 ${sonar_height/5}" rpy="${pi} ${pi} 0"/>
     </joint>
     <link name="sonar">
@@ -278,4 +278,5 @@
         </collision>
         <visual>
+            <origin xyz="0 0 0" rpy="${pi} ${pi} 0"/>
             <geometry>
                 <mesh filename="file://$(find turbopi_ros)/meshes/sonar.dae" scale="${mesh_scale}" />

Commit message: description/turbopi_core.xacro: Swap wheel mesh dae with stl
- Remove cascading origin changes

File: description/turbopi_core.xacro (robot description, xacro)
@@ -28,5 +28,5 @@
     <xacro:property name="wheel_radius" value="0.0325" />
     <xacro:property name="wheel_mass" value="0.0016" />
-    <xacro:property name="wheel_mesh_file" value="file://$(find turbopi_ros)/meshes/wheel.dae" />
+    <xacro:property name="wheel_mesh_file" value="file://$(find turbopi_ros)/meshes/wheel.stl" />
     <xacro:property name="wheel_offset_front" value="${-chassis_length/2 + 0.0372}" />
     <xacro:property name="wheel_offset_rear" value="${chassis_length/2 - 0.0305}" />
@@ -119,5 +119,5 @@
         <parent link="chassis"/>
         <child link="front_left_wheel"/>
-        <origin xyz="${wheel_offset_front} -${wheel_offset_side} -${wheel_zoffset}" rpy="${pi/2} ${pi/2} 0"/>
+        <origin xyz="${wheel_offset_front} -${wheel_offset_side} -${wheel_zoffset}" rpy="0 0 0"/>
         <axis xyz="0 0 1"/>
         <limit effort="${limit_effort}" velocity="${limit_velocity}"/>
@@ -130,5 +130,4 @@
         </collision>
         <visual>
-            <origin xyz="0 0 0" rpy="-${pi/2} 0 0"/>
             <geometry>
                 <mesh filename="${wheel_mesh_file}" scale="${mesh_scale}" />
@@ -144,5 +143,5 @@
         <parent link="chassis"/>
         <child link="front_right_wheel"/>
-        <origin xyz="${wheel_offset_front} ${wheel_offset_side} -${wheel_zoffset}" rpy="-${pi/2} ${pi/2} 0"/>
+        <origin xyz="${wheel_offset_front} ${wheel_offset_side} -${wheel_zoffset}" rpy="0 0 ${pi}"/>
         <axis xyz="0 0 -1"/>
         <limit effort="${limit_effort}" velocity="${limit_velocity}"/>
@@ -155,5 +154,4 @@
         </collision>
         <visual>
-            <origin xyz="0 0 0" rpy="-${pi/2} 0 0"/>
             <geometry>
                 <mesh filename="${wheel_mesh_file}" scale="${mesh_scale}" />
@@ -169,5 +167,5 @@
         <parent link="chassis"/>
         <child link="rear_left_wheel"/>
-        <origin xyz="${wheel_offset_rear} -${wheel_offset_side} -${wheel_zoffset}" rpy="${pi/2} ${pi/2} 0"/>
+        <origin xyz="${wheel_offset_rear} -${wheel_offset_side} -${wheel_zoffset}" rpy="0 0 0"/>
         <axis xyz="0 0 1"/>
         <limit effort="${limit_effort}" velocity="${limit_velocity}"/>
@@ -180,5 +178,4 @@
         </collision>
         <visual>
-            <origin xyz="0 0 0" rpy="-${pi/2} 0 0"/>
             <geometry>
                 <mesh filename="${wheel_mesh_file}" scale="${mesh_scale}" />
@@ -194,5 +191,5 @@
         <parent link="chassis"/>
         <child link="rear_right_wheel"/>
-        <origin xyz="${wheel_offset_rear} ${wheel_offset_side} -${wheel_zoffset}" rpy="-${pi/2} ${pi/2} 0"/>
+        <origin xyz="${wheel_offset_rear} ${wheel_offset_side} -${wheel_zoffset}" rpy="0 0 ${pi}"/>
         <axis xyz="0 0 -1"/>
         <limit effort="${limit_effort}" velocity="${limit_velocity}"/>
@@ -205,5 +202,4 @@
         </collision>
         <visual>
-            <origin xyz="0 0 0" rpy="-${pi/2} 0 0"/>
             <geometry>
                 <mesh filename="${wheel_mesh_file}" scale="${mesh_scale}" />

Commit message: description/turbopi_core.xacro: Swap chassis dae with stl

File: description/turbopi_core.xacro (robot description, xacro)
@@ -55,5 +55,5 @@
         <visual>
             <geometry>
-                <mesh filename="file://$(find turbopi_ros)/meshes/chassis.dae" scale="${mesh_scale}" />
+                <mesh filename="file://$(find turbopi_ros)/meshes/chassis.stl" scale="${mesh_scale}" />
             </geometry>
             <material name="white"/>

Commit message: description/turbopi_core.xacro: Swap space mesh dae with stl, add var

File: description/turbopi_core.xacro (robot description, xacro)
@@ -20,4 +20,5 @@
     <xacro:property name="sonar_height" value="0.0254" />
     <xacro:property name="sonar_width" value="0.0508" />
+    <xacro:property name="spacer_mesh_file" value="file://$(find turbopi_ros)/meshes/spacer.stl" />
     <xacro:property name="spacer_offset_front" value="0.0203" />
     <xacro:property name="spacer_offset_rear" value="${chassis_width - 0.0135}" />
@@ -71,5 +72,5 @@
         <visual>
             <geometry>
-                <mesh filename="file://$(find turbopi_ros)/meshes/spacer.dae" scale="${mesh_scale}" />
+                <mesh filename="${spacer_mesh_file}" scale="${mesh_scale}" />
             </geometry>
             <material name="brass"/>
@@ -84,5 +85,5 @@
         <visual>
             <geometry>
-                <mesh filename="file://$(find turbopi_ros)/meshes/spacer.dae" scale="${mesh_scale}" />
+                <mesh filename="${spacer_mesh_file}" scale="${mesh_scale}" />
             </geometry>
             <material name="brass"/>
@@ -97,5 +98,5 @@
         <visual>
             <geometry>
-                <mesh filename="file://$(find turbopi_ros)/meshes/spacer.dae" scale="${mesh_scale}" />
+                <mesh filename="${spacer_mesh_file}" scale="${mesh_scale}" />
             </geometry>
             <material name="brass"/>
@@ -110,5 +111,5 @@
         <visual>
             <geometry>
-                <mesh filename="file://$(find turbopi_ros)/meshes/spacer.dae" scale="${mesh_scale}" />
+                <mesh filename="${spacer_mesh_file}" scale="${mesh_scale}" />
             </geometry>
             <material name="brass"/>

Commit message: description/turbopi_core.xacro: Swap camera dae with stl

File: description/turbopi_core.xacro (robot description, xacro)
@@ -253,5 +253,5 @@
             <origin xyz="0 0 0" rpy="${pi} ${pi} 0"/>
             <geometry>
-                <mesh filename="file://$(find turbopi_ros)/meshes/camera.dae" scale="${mesh_scale}" />
+                <mesh filename="file://$(find turbopi_ros)/meshes/camera.stl" scale="${mesh_scale}" />
             </geometry>
             <material name="white"/>

Commit message: description/turbopi_core.xacro: Swap camera frame dae with stl

File: description/turbopi_core.xacro (robot description, xacro)
@@ -228,5 +228,5 @@
         <visual>
             <geometry>
-                <mesh filename="file://$(find turbopi_ros)/meshes/camera_frame.dae" scale="${mesh_scale}" />
+                <mesh filename="file://$(find turbopi_ros)/meshes/camera_frame.stl" scale="${mesh_scale}" />
             </geometry>
             <material name="white"/>

Commit message: description/turbopi_core.xacro: Swap sonar dae with stl

File: description/turbopi_core.xacro (robot description, xacro)
@@ -277,5 +277,5 @@
             <origin xyz="0 0 0" rpy="${pi} ${pi} 0"/>
             <geometry>
-                <mesh filename="file://$(find turbopi_ros)/meshes/sonar.dae" scale="${mesh_scale}" />
+                <mesh filename="file://$(find turbopi_ros)/meshes/sonar.stl" scale="${mesh_scale}" />
             </geometry>
             <material name="white"/>

Commit message: description/turbopi_core.xacro: Wrap camera & sonar in style macro
- Initial work to control 2d camera and sonar or other

File: description/turbopi_core.xacro (robot description, xacro)
@@ -212,77 +212,81 @@
         </xacro:inertial_cylinder>
     </link>
-    <!-- Camera frame turns left/right -->
-    <joint name="camera_frame_joint" type="revolute">
-        <parent link="chassis"/>
-        <child link="camera_frame"/>
-        <origin xyz="${-chassis_length/2 + 0.054} 0 ${chassis_height + 0.01}" rpy="0 0 0"/>
-        <limit lower="-1"  upper="1"  velocity="0.1"  effort="${limit_effort}"  />
-        <axis xyz="0 0 1"/>
-    </joint>
-    <link name="camera_frame">
-        <collision>
-            <geometry>
-                <box size="${camera_frame_length} ${camera_frame_width} ${camera_frame_height}"/>
-            </geometry>
-        </collision>
-        <visual>
-            <geometry>
-                <mesh filename="file://$(find turbopi_ros)/meshes/camera_frame.stl" scale="${mesh_scale}" />
-            </geometry>
-            <material name="white"/>
-        </visual>
-        <xacro:inertial_box mass="0.01" x="${camera_frame_length}" y="${camera_frame_width}" z="${camera_frame_height}">
-            <origin xyz="0 0 ${camera_frame_height/2}" rpy="0 0 0"/>
-        </xacro:inertial_box>
-    </link>
-    <!-- Camera angles up/down -->
-    <joint name="camera_joint" type="revolute">
-        <parent link="camera_frame"/>
-        <child link="camera"/>
-        <origin xyz="-0.015 0 ${camera_frame_height * 0.4}" rpy="${pi} ${pi} 0"/>
-        <limit lower="-0.5"  upper="1"  velocity="0.1"  effort="${limit_effort}"  />
-        <axis xyz="0 1 0"/>
-    </joint>
-    <link name="camera">
-        <collision>
-            <geometry>
-                <box size="${camera_length} ${camera_width} ${camera_height}"/>
-            </geometry>
-        </collision>
-        <visual>
-            <origin xyz="0 0 0" rpy="${pi} ${pi} 0"/>
-            <geometry>
-                <mesh filename="file://$(find turbopi_ros)/meshes/camera.stl" scale="${mesh_scale}" />
-            </geometry>
-            <material name="white"/>
-        </visual>
-        <xacro:inertial_box mass="0.01" x="${camera_length}" y="${camera_width}" z="${camera_height}">
-            <origin xyz="0 0 ${camera_height/2}" rpy="0 0 0"/>
-        </xacro:inertial_box>
-    </link>
-    <!-- Sonar -->
-    <joint name="sonar_joint" type="fixed">
-        <parent link="chassis"/>
-        <child link="sonar"/>
-        <axis xyz="0 0 1"/>
-        <origin xyz="-${chassis_length/2 - sonar_length*0.8} 0 ${sonar_height/5}" rpy="${pi} ${pi} 0"/>
-    </joint>
-    <link name="sonar">
-        <collision>
-            <geometry>
-                <box size="${sonar_length} ${sonar_width} ${sonar_height}"/>
-            </geometry>
-        </collision>
-        <visual>
-            <origin xyz="0 0 0" rpy="${pi} ${pi} 0"/>
-            <geometry>
-                <mesh filename="file://$(find turbopi_ros)/meshes/sonar.stl" scale="${mesh_scale}" />
-            </geometry>
-            <material name="white"/>
-        </visual>
-        <xacro:inertial_box mass="0.01" x="${sonar_length}" y="${sonar_width}" z="${sonar_height}">
-            <origin xyz="0 0 0" rpy="0 0 0"/>
-        </xacro:inertial_box>
-    </link>
+    <xacro:macro name="style" params="use_style">
+        <xacro:if value="${use_style == 'default'}">
+            <!-- Camera frame turns left/right -->
+            <joint name="camera_frame_joint" type="revolute">
+                <parent link="chassis"/>
+                <child link="camera_frame"/>
+                <origin xyz="${-chassis_length/2 + 0.054} 0 ${chassis_height + 0.01}" rpy="0 0 0"/>
+                <limit lower="-1"  upper="1"  velocity="0.1"  effort="${limit_effort}"  />
+                <axis xyz="0 0 1"/>
+            </joint>
+            <link name="camera_frame">
+                <collision>
+                    <geometry>
+                        <box size="${camera_frame_length} ${camera_frame_width} ${camera_frame_height}"/>
+                    </geometry>
+                </collision>
+                <visual>
+                    <geometry>
+                        <mesh filename="file://$(find turbopi_ros)/meshes/camera_frame.stl" scale="${mesh_scale}" />
+                    </geometry>
+                    <material name="white"/>
+                </visual>
+                <xacro:inertial_box mass="0.01" x="${camera_frame_length}" y="${camera_frame_width}" z="${camera_frame_height}">
+                    <origin xyz="0 0 ${camera_frame_height/2}" rpy="0 0 0"/>
+                </xacro:inertial_box>
+            </link>
+            <!-- Camera angles up/down -->
+            <joint name="camera_joint" type="revolute">
+                <parent link="camera_frame"/>
+                <child link="camera"/>
+                <origin xyz="-0.015 0 ${camera_frame_height * 0.4}" rpy="${pi} ${pi} 0"/>
+                <limit lower="-0.5"  upper="1"  velocity="0.1"  effort="${limit_effort}"  />
+                <axis xyz="0 1 0"/>
+            </joint>
+            <link name="camera">
+                <collision>
+                    <geometry>
+                        <box size="${camera_length} ${camera_width} ${camera_height}"/>
+                    </geometry>
+                </collision>
+                <visual>
+                    <origin xyz="0 0 0" rpy="${pi} ${pi} 0"/>
+                    <geometry>
+                        <mesh filename="file://$(find turbopi_ros)/meshes/camera.stl" scale="${mesh_scale}" />
+                    </geometry>
+                    <material name="white"/>
+                </visual>
+                <xacro:inertial_box mass="0.01" x="${camera_length}" y="${camera_width}" z="${camera_height}">
+                    <origin xyz="0 0 ${camera_height/2}" rpy="0 0 0"/>
+                </xacro:inertial_box>
+            </link>
+            <!-- Sonar -->
+            <joint name="sonar_joint" type="fixed">
+                <parent link="chassis"/>
+                <child link="sonar"/>
+                <axis xyz="0 0 1"/>
+                <origin xyz="-${chassis_length/2 - sonar_length*0.8} 0 ${sonar_height/5}" rpy="${pi} ${pi} 0"/>
+            </joint>
+            <link name="sonar">
+                <collision>
+                    <geometry>
+                        <box size="${sonar_length} ${sonar_width} ${sonar_height}"/>
+                    </geometry>
+                </collision>
+                <visual>
+                    <origin xyz="0 0 0" rpy="${pi} ${pi} 0"/>
+                    <geometry>
+                        <mesh filename="file://$(find turbopi_ros)/meshes/sonar.stl" scale="${mesh_scale}" />
+                    </geometry>
+                    <material name="white"/>
+                </visual>
+                <xacro:inertial_box mass="0.01" x="${sonar_length}" y="${sonar_width}" z="${sonar_height}">
+                    <origin xyz="0 0 0" rpy="0 0 0"/>
+                </xacro:inertial_box>
+            </link>
+        </xacro:if>
+    </xacro:macro>
     <!-- 360 Lidar -->
     <joint name="lidar_joint" type="fixed">
