Commit message: description/turbopi_core.xacro: Fix direction of chassis, camera, & sonar
- Flip the model around, changes per changes to the CAD files, robot
  was facing the wrong direction that required flipping the cameras around
- Proper orientation now, no excessive rpy transformations
- More changes/fixes to come per this correction

File: description/turbopi_core.xacro (robot description, xacro)
@@ -21,6 +21,6 @@
     <xacro:property name="sonar_width" value="0.0508" />
     <xacro:property name="spacer_mesh_file" value="file://$(find turbopi_ros)/meshes/spacer.stl" />
-    <xacro:property name="spacer_offset_front" value="0.0203" />
-    <xacro:property name="spacer_offset_rear" value="${chassis_width - 0.0135}" />
+    <xacro:property name="spacer_offset_front" value="-0.0203" />
+    <xacro:property name="spacer_offset_rear" value="${-chassis_width + 0.0135}" />
     <xacro:property name="spacer_offset_side" value="${chassis_width/2 - 0.0138}" />
     <xacro:property name="spacer_offset_height" value="0.015" />
@@ -218,5 +218,5 @@
                 <parent link="chassis"/>
                 <child link="camera_frame"/>
-                <origin xyz="${-chassis_length/2 + 0.054} 0 ${chassis_height + 0.01}" rpy="0 0 0"/>
+                <origin xyz="${chassis_length/2 - 0.054} 0 ${chassis_height + 0.01}" rpy="0 0 0"/>
                 <limit lower="-1"  upper="1"  velocity="0.1"  effort="${limit_effort}"  />
                 <axis xyz="0 0 1"/>
@@ -242,5 +242,5 @@
                 <parent link="camera_frame"/>
                 <child link="camera"/>
-                <origin xyz="-0.015 0 ${camera_frame_height * 0.4}" rpy="${pi} ${pi} 0"/>
+                <origin xyz="0.015 0 ${camera_frame_height * 0.4}" rpy="0 0 0"/>
                 <limit lower="-0.5"  upper="1"  velocity="0.1"  effort="${limit_effort}"  />
                 <axis xyz="0 1 0"/>
@@ -253,5 +253,5 @@
                 </collision>
                 <visual>
-                    <origin xyz="0 0 0" rpy="${pi} ${pi} 0"/>
+                    <origin xyz="0 0 0" rpy="0 0 0"/>
                     <geometry>
                         <mesh filename="file://$(find turbopi_ros)/meshes/camera.stl" scale="${mesh_scale}" />
@@ -268,5 +268,5 @@
                 <child link="sonar"/>
                 <axis xyz="0 0 1"/>
-                <origin xyz="-${chassis_length/2 - sonar_length*0.8} 0 ${sonar_height/5}" rpy="${pi} ${pi} 0"/>
+                <origin xyz="${chassis_length/2 - sonar_length*0.8} 0 ${sonar_height/5}" rpy="0 0 0"/>
             </joint>
             <link name="sonar">
@@ -277,5 +277,5 @@
                 </collision>
                 <visual>
-                    <origin xyz="0 0 0" rpy="${pi} ${pi} 0"/>
+                    <origin xyz="0 0 0" rpy="0 0 0"/>
                     <geometry>
                         <mesh filename="file://$(find turbopi_ros)/meshes/sonar.stl" scale="${mesh_scale}" />
@@ -294,5 +294,5 @@
         <child link="lidar"/>
         <axis xyz="0 0 1"/>
-        <origin xyz="${lidar_length/2 - 0.01} 0 0.0725" rpy="0 0 0"/>
+        <origin xyz="${-lidar_length/2 + 0.01} 0 0.0725" rpy="0 0 0"/>
     </joint>
     <link name="lidar">

Commit message: description/turbopi_core.xacro: Fix wheel rotation axis, broken by changes

File: description/turbopi_core.xacro (robot description, xacro)
@@ -121,5 +121,5 @@
         <child link="front_left_wheel"/>
         <origin xyz="${wheel_offset_front} -${wheel_offset_side} -${wheel_zoffset}" rpy="0 0 0"/>
-        <axis xyz="0 0 1"/>
+        <axis xyz="0 1 0"/>
         <limit effort="${limit_effort}" velocity="${limit_velocity}"/>
     </joint>
@@ -145,5 +145,5 @@
         <child link="front_right_wheel"/>
         <origin xyz="${wheel_offset_front} ${wheel_offset_side} -${wheel_zoffset}" rpy="0 0 ${pi}"/>
-        <axis xyz="0 0 -1"/>
+        <axis xyz="0 -1 0"/>
         <limit effort="${limit_effort}" velocity="${limit_velocity}"/>
     </joint>
@@ -169,5 +169,5 @@
         <child link="rear_left_wheel"/>
         <origin xyz="${wheel_offset_rear} -${wheel_offset_side} -${wheel_zoffset}" rpy="0 0 0"/>
-        <axis xyz="0 0 1"/>
+        <axis xyz="0 1 0"/>
         <limit effort="${limit_effort}" velocity="${limit_velocity}"/>
     </joint>
@@ -193,5 +193,5 @@
         <child link="rear_right_wheel"/>
         <origin xyz="${wheel_offset_rear} ${wheel_offset_side} -${wheel_zoffset}" rpy="0 0 ${pi}"/>
-        <axis xyz="0 0 -1"/>
+        <axis xyz="0 -1 0"/>
         <limit effort="${limit_effort}" velocity="${limit_velocity}"/>
     </joint>

Commit message: description/turbopi_core.xacro: Initial conditional depth camera

File: description/turbopi_core.xacro (robot description, xacro)
@@ -13,4 +13,7 @@
     <xacro:property name="chassis_height" value="0.04" />
     <xacro:property name="chassis_width" value="0.094" />
+    <xacro:property name="depth_camera_length" value="0.165" />
+    <xacro:property name="depth_camera_height" value="0.40" />
+    <xacro:property name="depth_camera_width" value="0.48" />
     <xacro:property name="lidar_length" value="0.12954" />
     <xacro:property name="lidar_height" value="0.07874" />
@@ -288,4 +291,30 @@
             </link>
         </xacro:if>
+        <xacro:if value="${use_style == 'depth'}">
+            <!-- 3D Depth Camera -->
+            <joint name="depth_camera_joint" type="fixed">
+                <parent link="chassis"/>
+                <child link="depth_camera"/>
+                <axis xyz="0 0 1"/>
+                <origin xyz="${chassis_length/2 - 0.054} 0 ${chassis_height}" rpy="0 0 0"/>
+            </joint>
+            <link name="depth_camera">
+                <!-- Causes floating? -->
+                <!-- <collision>
+                    <geometry>
+                        <box size="${depth_camera_length} ${depth_camera_width} ${depth_camera_height}"/>
+                    </geometry>
+                </collision> -->
+                <visual>
+                    <geometry>
+                        <mesh filename="file://$(find turbopi_ros)/meshes/astra_s_depth_camera.stl" scale="${mesh_scale}" />
+                    </geometry>
+                    <material name="white"/>
+                </visual>
+                <xacro:inertial_box mass="0.02" x="${depth_camera_length}" y="${depth_camera_width}" z="${depth_camera_height}">
+                    <origin xyz="0 0 ${depth_camera_height/2}" rpy="0 0 0"/>
+                </xacro:inertial_box>
+            </link>
+        </xacro:if>
     </xacro:macro>
     <!-- 360 Lidar -->

Commit message: description/turbopi_core.xacro: Fix wheel axis and rotation

File: description/turbopi_core.xacro (robot description, xacro)
@@ -123,6 +123,6 @@
         <parent link="chassis"/>
         <child link="front_left_wheel"/>
-        <origin xyz="${wheel_offset_front} -${wheel_offset_side} -${wheel_zoffset}" rpy="0 0 0"/>
-        <axis xyz="0 1 0"/>
+        <origin xyz="${wheel_offset_front} -${wheel_offset_side} -${wheel_zoffset}" rpy="${pi/2} 0 0"/>
+        <axis xyz="0 0 -1"/>
         <limit effort="${limit_effort}" velocity="${limit_velocity}"/>
     </joint>
@@ -147,6 +147,6 @@
         <parent link="chassis"/>
         <child link="front_right_wheel"/>
-        <origin xyz="${wheel_offset_front} ${wheel_offset_side} -${wheel_zoffset}" rpy="0 0 ${pi}"/>
-        <axis xyz="0 -1 0"/>
+        <origin xyz="${wheel_offset_front} ${wheel_offset_side} -${wheel_zoffset}" rpy="${pi/2} 0 ${pi}"/>
+        <axis xyz="0 0 1"/>
         <limit effort="${limit_effort}" velocity="${limit_velocity}"/>
     </joint>
@@ -171,6 +171,6 @@
         <parent link="chassis"/>
         <child link="rear_left_wheel"/>
-        <origin xyz="${wheel_offset_rear} -${wheel_offset_side} -${wheel_zoffset}" rpy="0 0 0"/>
-        <axis xyz="0 1 0"/>
+        <origin xyz="${wheel_offset_rear} -${wheel_offset_side} -${wheel_zoffset}" rpy="${pi/2} 0 0"/>
+        <axis xyz="0 0 -1"/>
         <limit effort="${limit_effort}" velocity="${limit_velocity}"/>
     </joint>
@@ -195,6 +195,6 @@
         <parent link="chassis"/>
         <child link="rear_right_wheel"/>
-        <origin xyz="${wheel_offset_rear} ${wheel_offset_side} -${wheel_zoffset}" rpy="0 0 ${pi}"/>
-        <axis xyz="0 -1 0"/>
+        <origin xyz="${wheel_offset_rear} ${wheel_offset_side} -${wheel_zoffset}" rpy="${pi/2} 0 ${pi}"/>
+        <axis xyz="0 0 1"/>
         <limit effort="${limit_effort}" velocity="${limit_velocity}"/>
     </joint>

Commit message: description/turbopi_core.xacro: Move sonar sensor out of conditional
- The lights and look will be used for depth camera, in addition to 2d
  even if the sonar data itself is not used.

File: description/turbopi_core.xacro (robot description, xacro)
@@ -266,28 +266,4 @@
                 </xacro:inertial_box>
             </link>
-            <!-- Sonar -->
-            <joint name="sonar_joint" type="fixed">
-                <parent link="chassis"/>
-                <child link="sonar"/>
-                <axis xyz="0 0 1"/>
-                <origin xyz="${chassis_length/2 - sonar_length*0.8} 0 ${sonar_height/5}" rpy="0 0 0"/>
-            </joint>
-            <link name="sonar">
-                <collision>
-                    <geometry>
-                        <box size="${sonar_length} ${sonar_width} ${sonar_height}"/>
-                    </geometry>
-                </collision>
-                <visual>
-                    <origin xyz="0 0 0" rpy="0 0 0"/>
-                    <geometry>
-                        <mesh filename="file://$(find turbopi_ros)/meshes/sonar.stl" scale="${mesh_scale}" />
-                    </geometry>
-                    <material name="white"/>
-                </visual>
-                <xacro:inertial_box mass="0.01" x="${sonar_length}" y="${sonar_width}" z="${sonar_height}">
-                    <origin xyz="0 0 0" rpy="0 0 0"/>
-                </xacro:inertial_box>
-            </link>
         </xacro:if>
         <xacro:if value="${use_style == 'depth'}">
@@ -318,4 +294,28 @@
         </xacro:if>
     </xacro:macro>
+    <!-- Sonar -->
+    <joint name="sonar_joint" type="fixed">
+        <parent link="chassis"/>
+        <child link="sonar"/>
+        <axis xyz="0 0 1"/>
+        <origin xyz="${chassis_length/2 - sonar_length*0.8} 0 ${sonar_height/5}" rpy="0 0 0"/>
+    </joint>
+    <link name="sonar">
+        <collision>
+            <geometry>
+                <box size="${sonar_length} ${sonar_width} ${sonar_height}"/>
+            </geometry>
+        </collision>
+        <visual>
+            <origin xyz="0 0 0" rpy="0 0 0"/>
+            <geometry>
+                <mesh filename="file://$(find turbopi_ros)/meshes/sonar.stl" scale="${mesh_scale}" />
+            </geometry>
+            <material name="white"/>
+        </visual>
+        <xacro:inertial_box mass="0.01" x="${sonar_length}" y="${sonar_width}" z="${sonar_height}">
+            <origin xyz="0 0 0" rpy="0 0 0"/>
+        </xacro:inertial_box>
+    </link>
     <!-- 360 Lidar -->
     <joint name="lidar_joint" type="fixed">

Commit message: description/turbopi_core.xacro: Rotate wheels, correct diretion side, etc
- Final reminent from flipping the chassis around and correcting CAD
  wheel alignment to reduce math, and orgin transformations

File: description/turbopi_core.xacro (robot description, xacro)
@@ -33,6 +33,6 @@
     <xacro:property name="wheel_mass" value="0.0016" />
     <xacro:property name="wheel_mesh_file" value="file://$(find turbopi_ros)/meshes/wheel.stl" />
-    <xacro:property name="wheel_offset_front" value="${-chassis_length/2 + 0.0372}" />
-    <xacro:property name="wheel_offset_rear" value="${chassis_length/2 - 0.0305}" />
+    <xacro:property name="wheel_offset_front" value="${chassis_length/2 - 0.0305}" />
+    <xacro:property name="wheel_offset_rear" value="${-chassis_length/2 + 0.0372}" />
     <xacro:property name="wheel_offset_side" value="${wheel_length/2 + chassis_width/2 + wheel_gap}" />
     <xacro:property name="wheel_zoffset" value="${chassis_height/2 + 0.0064}" />
@@ -123,9 +123,33 @@
         <parent link="chassis"/>
         <child link="front_left_wheel"/>
+        <origin xyz="${wheel_offset_front} ${wheel_offset_side} -${wheel_zoffset}" rpy="${pi/2} 0 ${pi}"/>
+        <axis xyz="0 0 1"/>
+        <limit effort="${limit_effort}" velocity="${limit_velocity}"/>
+    </joint>
+    <link name="front_left_wheel">
+        <collision>
+            <geometry>
+                <cylinder length="${wheel_length * collision_multiplier}" radius="${wheel_radius}" />
+            </geometry>
+        </collision>
+        <visual>
+            <geometry>
+                <mesh filename="${wheel_mesh_file}" scale="${mesh_scale}" />
+            </geometry>
+            <material name="yellow"/>
+        </visual>
+        <xacro:inertial_cylinder mass="${wheel_mass}" length="${wheel_length}" radius="${wheel_radius}">
+            <origin xyz="0 0 0" rpy="0 0 0"/>
+        </xacro:inertial_cylinder>
+    </link>
+    <!-- Front Right Wheel -->
+    <joint name="front_right_wheel_joint" type="continuous">
+        <parent link="chassis"/>
+        <child link="front_right_wheel"/>
         <origin xyz="${wheel_offset_front} -${wheel_offset_side} -${wheel_zoffset}" rpy="${pi/2} 0 0"/>
         <axis xyz="0 0 -1"/>
         <limit effort="${limit_effort}" velocity="${limit_velocity}"/>
     </joint>
-    <link name="front_left_wheel">
+    <link name="front_right_wheel">
         <collision>
             <geometry>
@@ -143,13 +167,13 @@
         </xacro:inertial_cylinder>
     </link>
-    <!-- Front Right Wheel -->
-    <joint name="front_right_wheel_joint" type="continuous">
-        <parent link="chassis"/>
-        <child link="front_right_wheel"/>
-        <origin xyz="${wheel_offset_front} ${wheel_offset_side} -${wheel_zoffset}" rpy="${pi/2} 0 ${pi}"/>
+    <!-- Rear Left Wheel -->
+    <joint name="rear_left_wheel_joint" type="continuous">
+        <parent link="chassis"/>
+        <child link="rear_left_wheel"/>
+        <origin xyz="${wheel_offset_rear} ${wheel_offset_side} -${wheel_zoffset}" rpy="${pi/2} 0 ${pi}"/>
         <axis xyz="0 0 1"/>
         <limit effort="${limit_effort}" velocity="${limit_velocity}"/>
     </joint>
-    <link name="front_right_wheel">
+    <link name="rear_left_wheel">
         <collision>
             <geometry>
@@ -167,34 +191,10 @@
         </xacro:inertial_cylinder>
     </link>
-    <!-- Rear Left Wheel -->
-    <joint name="rear_left_wheel_joint" type="continuous">
-        <parent link="chassis"/>
-        <child link="rear_left_wheel"/>
+    <!-- Rear Right Wheel -->
+    <joint name="rear_right_wheel_joint" type="continuous">
+        <parent link="chassis"/>
+        <child link="rear_right_wheel"/>
         <origin xyz="${wheel_offset_rear} -${wheel_offset_side} -${wheel_zoffset}" rpy="${pi/2} 0 0"/>
         <axis xyz="0 0 -1"/>
-        <limit effort="${limit_effort}" velocity="${limit_velocity}"/>
-    </joint>
-    <link name="rear_left_wheel">
-        <collision>
-            <geometry>
-                <cylinder length="${wheel_length * collision_multiplier}" radius="${wheel_radius}" />
-            </geometry>
-        </collision>
-        <visual>
-            <geometry>
-                <mesh filename="${wheel_mesh_file}" scale="${mesh_scale}" />
-            </geometry>
-            <material name="yellow"/>
-        </visual>
-        <xacro:inertial_cylinder mass="${wheel_mass}" length="${wheel_length}" radius="${wheel_radius}">
-            <origin xyz="0 0 0" rpy="0 0 0"/>
-        </xacro:inertial_cylinder>
-    </link>
-    <!-- Rear Right Wheel -->
-    <joint name="rear_right_wheel_joint" type="continuous">
-        <parent link="chassis"/>
-        <child link="rear_right_wheel"/>
-        <origin xyz="${wheel_offset_rear} ${wheel_offset_side} -${wheel_zoffset}" rpy="${pi/2} 0 ${pi}"/>
-        <axis xyz="0 0 1"/>
         <limit effort="${limit_effort}" velocity="${limit_velocity}"/>
     </joint>

Commit message: description/turbopi_core.xacro: Make lidar optional via use_lidar

File: description/turbopi_core.xacro (robot description, xacro)
@@ -312,25 +312,29 @@
     </link>
     <!-- 360 Lidar -->
-    <joint name="lidar_joint" type="fixed">
-        <parent link="chassis"/>
-        <child link="lidar"/>
-        <axis xyz="0 0 1"/>
-        <origin xyz="${-lidar_length/2 + 0.01} 0 0.0725" rpy="0 0 0"/>
-    </joint>
-    <link name="lidar">
-        <collision>
-            <geometry>
-                <box size="${lidar_length} ${lidar_width} ${lidar_height}"/>
-            </geometry>
-        </collision>
-        <visual>
-            <geometry>
-                <mesh filename="file://$(find turbopi_ros)/meshes/rplidar.dae" scale="1 1 1" />
-            </geometry>
-            <material name="black"/>
-        </visual>
-        <xacro:inertial_box mass="0.01" x="${lidar_length}" y="${lidar_width}" z="${chassis_height}">
-            <origin xyz="0 0 0" rpy="0 0 0"/>
-        </xacro:inertial_box>
-    </link>
+    <xacro:macro name="lidar" params="use_lidar">
+        <xacro:if value="${use_lidar == 'lidar'}">
+            <joint name="lidar_joint" type="fixed">
+                <parent link="chassis"/>
+                <child link="lidar"/>
+                <axis xyz="0 0 1"/>
+                <origin xyz="${-lidar_length/2 + 0.01} 0 0.0725" rpy="0 0 0"/>
+            </joint>
+            <link name="lidar">
+                <collision>
+                    <geometry>
+                        <box size="${lidar_length} ${lidar_width} ${lidar_height}"/>
+                    </geometry>
+                </collision>
+                <visual>
+                    <geometry>
+                        <mesh filename="file://$(find turbopi_ros)/meshes/rplidar.dae" scale="1 1 1" />
+                    </geometry>
+                    <material name="black"/>
+                </visual>
+                <xacro:inertial_box mass="0.01" x="${lidar_length}" y="${lidar_width}" z="${chassis_height}">
+                    <origin xyz="0 0 0" rpy="0 0 0"/>
+                </xacro:inertial_box>
+            </link>
+        </xacro:if>
+    </xacro:macro>
 </robot>
