Commit message: description/gazebo_plugins.xacro: Added gazebo plugin version variable
- Issues with gazebo 8 stack, requiring use of gazebo 6 still :(

File: description/gazebo_plugins.xacro (robot description, xacro)
@@ -100,30 +100,32 @@
         </sensor>
     </gazebo>
-    <gazebo>
-        <plugin filename="libgz_ros2_control-system.so" name="gz_ros2_control::GazeboSimROS2ControlPlugin">
-            <robot_param>robot_description</robot_param>
-            <robot_param_node>robot_state_publisher</robot_param_node>
-            <parameters>$(find turbopi_ros)/config/turbopi_controllers.yaml</parameters>
-        </plugin>
-        <plugin filename="libgz-sim8-diff-drive-system.so" name="gz::sim::systems::DiffDrive">
-            <left_joint>front_left_wheel_joint</left_joint>
-            <left_joint>rear_left_wheel_joint</left_joint>
-            <right_joint>front_right_wheel_joint</right_joint>
-            <right_joint>rear_right_wheel_joint</right_joint>
-            <wheel_separation>1</wheel_separation>
-            <wheel_radius>0.192</wheel_radius>
-            <wheels_per_side>2</wheels_per_side>
-            <odom_publish_frequency>10</odom_publish_frequency>
-            <odom_frame_id>odom</odom_frame_id>
-            <base_frame_id> base_link</base_frame_id>
-            <enable_odom_tf>true</enable_odom_tf>
-            <use_stamped_vel>false</use_stamped_vel>
-            <topic>cmd_vel</topic>
-            <odom_topic>odom</odom_topic>
-            <tf_topic>tf</tf_topic>
-        </plugin>
-        <plugin filename="libgz-sim8-sensors-system.so" name="gz::sim::systems::Sensors">
-            <render_engine>ogre2</render_engine>
-        </plugin>
-    </gazebo>
+    <xacro:macro name="plugins" params="use_version">
+        <gazebo>
+            <plugin filename="libgz_ros2_control-system.so" name="gz_ros2_control::GazeboSimROS2ControlPlugin">
+                <robot_param>robot_description</robot_param>
+                <robot_param_node>robot_state_publisher</robot_param_node>
+                <parameters>$(find turbopi_ros)/config/turbopi_controllers.yaml</parameters>
+            </plugin>
+            <plugin filename="libgz-sim${use_version}-diff-drive-system.so" name="gz::sim::systems::DiffDrive">
+                <left_joint>front_left_wheel_joint</left_joint>
+                <left_joint>rear_left_wheel_joint</left_joint>
+                <right_joint>front_right_wheel_joint</right_joint>
+                <right_joint>rear_right_wheel_joint</right_joint>
+                <wheel_separation>1</wheel_separation>
+                <wheel_radius>0.192</wheel_radius>
+                <wheels_per_side>2</wheels_per_side>
+                <odom_publish_frequency>10</odom_publish_frequency>
+                <odom_frame_id>odom</odom_frame_id>
+                <base_frame_id> base_link</base_frame_id>
+                <enable_odom_tf>true</enable_odom_tf>
+                <use_stamped_vel>false</use_stamped_vel>
+                <topic>cmd_vel</topic>
+                <odom_topic>odom</odom_topic>
+                <tf_topic>tf</tf_topic>
+            </plugin>
+            <plugin filename="libgz-sim${use_version}-sensors-system.so" name="gz::sim::systems::Sensors">
+                <render_engine>ogre2</render_engine>
+            </plugin>
+        </gazebo>
+    </xacro:macro>
 </robot>

Commit message: description/gazebo_plugins.xacro: Add joint state publisher plugin
- Switch from ros joint state publisher to gazebo

File: description/gazebo_plugins.xacro (robot description, xacro)
@@ -120,4 +120,11 @@
                 <tf_topic>tf</tf_topic>
             </plugin>
+            <plugin filename="libgz-sim-joint-state-publisher-system.so" name="gz::sim::systems::JointStatePublisher">
+                <topic>/joint_states</topic>
+                <joint>front_left_wheel_joint</joint>
+                <joint>front_right_wheel_joint</joint>
+                <joint>rear_left_wheel_joint</joint>
+                <joint>rear_right_wheel_joint</joint>
+            </plugin>
             <plugin filename="libgz-sim${use_version}-sensors-system.so" name="gz::sim::systems::Sensors">
                 <render_engine>ogre2</render_engine>

Commit message: description/gazebo_plugins.xacro: Initial support for mecanum or diff drive

File: description/gazebo_plugins.xacro (robot description, xacro)
@@ -100,24 +100,42 @@
         </sensor>
     </gazebo>
-    <xacro:macro name="plugins" params="use_version">
+    <xacro:macro name="plugins" params="use_drive use_version">
         <gazebo>
             <plugin filename="libgz_ros2_control-system.so" name="gz_ros2_control::GazeboSimROS2ControlPlugin">
                 <parameters>$(find turbopi_ros)/config/turbopi_controllers.yaml</parameters>
             </plugin>
-            <plugin filename="libgz-sim${use_version}-diff-drive-system.so" name="gz::sim::systems::DiffDrive">
-                <left_joint>front_left_wheel_joint</left_joint>
-                <left_joint>rear_left_wheel_joint</left_joint>
-                <right_joint>front_right_wheel_joint</right_joint>
-                <right_joint>rear_right_wheel_joint</right_joint>
-                <wheel_separation>1</wheel_separation>
-                <wheel_radius>0.192</wheel_radius>
-                <wheels_per_side>2</wheels_per_side>
-                <odom_publish_frequency>10</odom_publish_frequency>
-                <enable_odom_tf>true</enable_odom_tf>
-                <use_stamped_vel>false</use_stamped_vel>
-                <topic>cmd_vel</topic>
-                <odom_topic>odom</odom_topic>
-                <tf_topic>tf</tf_topic>
-            </plugin>
+            <xacro:if value="${use_drive == 'diff'}">
+                <plugin filename="libgz-sim${use_version}-diff-drive-system.so" name="gz::sim::systems::DiffDrive">
+                    <left_joint>front_left_wheel_joint</left_joint>
+                    <left_joint>rear_left_wheel_joint</left_joint>
+                    <right_joint>front_right_wheel_joint</right_joint>
+                    <right_joint>rear_right_wheel_joint</right_joint>
+                    <wheel_separation>1</wheel_separation>
+                    <wheel_radius>0.192</wheel_radius>
+                    <wheels_per_side>2</wheels_per_side>
+                    <odom_publish_frequency>10</odom_publish_frequency>
+                    <enable_odom_tf>true</enable_odom_tf>
+                    <use_stamped_vel>false</use_stamped_vel>
+                    <topic>cmd_vel</topic>
+                    <odom_topic>odom</odom_topic>
+                    <tf_topic>tf</tf_topic>
+                </plugin>
+            </xacro:if>
+            <xacro:if value="${use_drive == 'mecanum'}">
+                <plugin filename="libgz-sim${use_version}-mecanum-drive-system.so" name="gz::sim::systems::MecanumDrive">
+                    <front_left_joint>front_left_wheel_joint</front_left_joint>
+                    <rear_left_joint>rear_left_wheel_joint</rear_left_joint>
+                    <front_right_joint>front_right_wheel_joint</front_right_joint>
+                    <rear_right_joint>rear_right_wheel_joint</rear_right_joint>
+                    <wheel_separation>1</wheel_separation>
+                    <wheel_radius>0.192</wheel_radius>
+                    <odom_publish_frequency>10</odom_publish_frequency>
+                    <enable_odom_tf>true</enable_odom_tf>
+                    <use_stamped_vel>false</use_stamped_vel>
+                    <topic>cmd_vel</topic>
+                    <odom_topic>odom</odom_topic>
+                    <tf_topic>tf</tf_topic>
+                </plugin>
+            </xacro:if>
             <plugin filename="libgz-sim-joint-state-publisher-system.so" name="gz::sim::systems::JointStatePublisher">
                 <topic>/joint_states</topic>
